File: StealthPad/StealthPad.kicad_pcb (KiCad board)
At the start: 2 copper layers, 100 parts, among them J1 USB_C_Receptacle_USB2.0, K00 ESC, K01 7, K02 8, K03 9, K04 0, K05 -, K06 =, K10 1, K11 2, K12 3, K13 4, K14 5, K15 6, K20 CAPS, K21 TAB, K22 Q, K23 W, K24 E, K25 R, K26 T, K31 LALT, K32 A, K33 S, K34 D, K35 F, K36 G, K41 LSHIFT, K44 V, K45 B, K46 P, K51 LCTRL, K55 C, K56 SPACE, SW1 SW_PUSH, U1 W25Q128JVS, U2 USBLC6-2SC6, U4 XC6206PxxxMR, Y1 XTAL_GND

Commit message: Just a lil updatin'
Parts:
- added U3: RP2040, RP2040-QFN:RP2040-QFN-56, B.Cu at (115.0, 177.1)
- C1, C10, C11, C12, C13, C14, C15, C2, C3, C4, C5, C6, C7, C8, C9, D00, D01, D02, D03, D04, D05, D06, D10, D11, D12, D13, D14, D15, D20, D21, D22, D23, D24, D25, D26, D31, D32, D33, D34, D35, D36, D41, D44, D45, D46, D51, D55, D56, F1, FID3, FID4, J1, K00, K01, K02, K03, K04, K05, K06, K10, K11, K12, K13, K14, K15, K20, K21, K22, K23, K24, K25, K26, K31, K32, K33, K34, K35, K36, K41, K44, K45, K46, K51, K55, K56, R1, R2, R3, R4, R5, R6, R7, SW1, U1, U2, U4, Y1: moved to B.Cu
- C16: footprint Diode_SMD:D_SOD-123 -> Capacitor_SMD:C_0603_1608Metric; moved to B.Cu
- moved FID3 323.8 mm to (60.3, 192.3), turned to 180 degrees
- moved FID1 307.9 mm to (44.9, 82.0)
- moved D20 289.1 mm to (53.0, 134.0), turned to 90 degrees
- moved R2 285.7 mm to (111.5, 182.4)
- moved Y1 280.8 mm to (119.0, 192.0), turned to 180 degrees
- moved C3 272.8 mm to (114.9, 191.9), turned to 90 degrees
- moved C4 269.8 mm to (112.0, 170.3), turned to -90 degrees
- moved U4 265.9 mm to (105.4, 159.6), turned to 90 degrees
- moved K21 256.8 mm to (66.1, 129.3), turned to 180 degrees
- moved D10 252.9 mm to (71.0, 110.1), turned to 90 degrees
- moved C15 248.7 mm to (104.6, 156.7), turned to 180 degrees
- moved K11 247.8 mm to (83.8, 104.1), turned to -174.45 degrees
- moved C6 247.3 mm to (112.5, 185.8), turned to -90 degrees
- moved C11 243.0 mm to (106.5, 181.4), turned to -135 degrees
- moved C8 242.5 mm to (110.1, 170.3), turned to 90 degrees
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Connections:
- R2 pad 2: RESET -> Net-(R2-Pad2)
- Y1 pad 2: /XTAL_0 -> GND
- Y1 pad 3: GND -> /XTAL_0
- Y1 pad 4: (no net) -> GND
Routing:
- net ROW4: track 0.00 -> 151.7 mm
- net ROW2: track 0.00 -> 137.3 mm, vias 0 -> 2
- net COL5: track 0.00 -> 129.0 mm, vias 0 -> 6
- net ROW5: track 0.00 -> 124.3 mm
- net ROW0: track 0.00 -> 122.0 mm, vias 0 -> 2
- net COL6: track 0.00 -> 120.8 mm, vias 0 -> 5
- net ROW3: track 0.00 -> 118.3 mm, vias 0 -> 2
- net D_N: track 0.00 -> 103.2 mm
- net D_P: track 0.00 -> 103.2 mm
- net +5V: track 0.00 -> 102.2 mm
- net ROW1: track 0.00 -> 100.5 mm, vias 0 -> 4
- net +3V3: track 0.00 -> 63.7 mm, vias 0 -> 4
- net GND: track 0.00 -> 42.5 mm, vias 0 -> 19
- net CS: track 0.00 -> 31.6 mm
- net SD1: track 0.00 -> 27.8 mm
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- added copper zone on B.Cu, net +1V1
- added copper zone on B.Cu, net +3V3
- added copper zone on B.Cu, net GND
- added copper zone on F.Cu, net GND

Commit message: WIP Updates
Parts:
- removed FID1, FID2, FID3, FID4: Fiducial, Fiducial:Fiducial_0.75mm_Mask1.5mm
- added REF**: JLC-PartNumberMarker, MatchstickWorks:JLC-PartNumberMarker, F.Cu at (92.5, 160.1)
- added REF**: MW-Logo-Silk_6.25mm-dia, MatchstickWorks:MW-Logo-Silk_6.25mm-dia, F.Cu at (127.9, 65.7)
- added SW2: SW_PUSH, Keeb_Parts:SW_TACTILE_SMD, B.Cu at (133.3, 170.1)
- C1: value 100nF -> 22pF
- C3: value 22pF -> 100nF
- moved C3 26.9 mm to (120.7, 165.7), turned to 180 degrees
- moved C1 26.4 mm to (123.2, 191.9), turned to -90 degrees
- moved C2 8.33 mm to (114.9, 191.9), turned to 90 degrees
- moved R3 5.06 mm to (110.9, 69.8)
- moved F1 5.06 mm to (108.6, 72.5)
- moved R4 5.06 mm to (116.7, 69.8)
- moved U2 5.06 mm to (113.8, 70.4)
- moved J1 5.06 mm to (113.8, 61.5)
Connections:
- C1 pad 1: +3V3 -> GND
- C1 pad 2: GND -> XTAL_IN
- C2 pad 2: XTAL_IN -> /XTAL_0
- C3 pad 1: GND -> +3V3
- C3 pad 2: /XTAL_0 -> GND
- U3 pad 2: COL0 -> unconnected-(U3-Pad2)
- U3 pad 3: COL1 -> unconnected-(U3-Pad3)
- U3 pad 34: ROW3 -> COL1
- U3 pad 35: ROW2 -> COL0
- U3 pad 36: ROW1 -> COL2
- U3 pad 37: ROW0 -> COL3
- U3 pad 38: unconnected-(U3-Pad38) -> ROW0
- U3 pad 39: unconnected-(U3-Pad39) -> ROW1
- U3 pad 4: COL2 -> unconnected-(U3-Pad4)
- U3 pad 40: unconnected-(U3-Pad40) -> ROW2
- U3 pad 41: unconnected-(U3-Pad41) -> ROW3
- U3 pad 5: COL3 -> unconnected-(U3-Pad5)
Routing:
- net COL1: track 0.00 -> 193.6 mm, vias 0 -> 7
- net COL0: track 0.00 -> 175.8 mm, vias 0 -> 6
- net ROW0: track 122.0 -> 268.5 mm
- net COL4: track 0.00 -> 144.2 mm, vias 0 -> 6
- net COL2: track 0.00 -> 127.1 mm, vias 0 -> 5
- net COL3: track 0.00 -> 124.9 mm, vias 0 -> 9
- net ROW1: track 100.5 -> 219.3 mm
- net ROW2: track 137.3 -> 217.6 mm
- net COL6: track 120.8 -> 190.5 mm, vias 5 -> 7
- net ROW3: track 118.3 -> 166.7 mm
- net Net-(R2-Pad2): track 2.22 -> 41.7 mm, vias 0 -> 2
- net ROW4: track 151.7 -> 190.8 mm
- net ROW5: track 124.3 -> 161.5 mm, vias 0 -> 2
- net COL5: track 129.0 -> 164.7 mm, vias 6 -> 8
- net D_N: track 103.2 -> 98.1 mm
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Other:
- board outline added: 165 x 147.2 mm
- board text added: "MatchstickWorks StealthPad v0.1"
