File: StealthPad/StealthPad.kicad_sch (KiCad schematic)
At the start: 72 parts, among them J1 USB_C_Receptacle_USB2.0, K00 KEYSW, K01 KEYSW, K02 KEYSW, K03 KEYSW, K04 KEYSW, K05 KEYSW, K06 KEYSW, K10 KEYSW, K11 KEYSW, K12 KEYSW, K13 KEYSW, K14 KEYSW, K15 KEYSW, K20 KEYSW, K21 KEYSW, K22 KEYSW, K23 KEYSW, K24 KEYSW, K25 KEYSW, K26 KEYSW, K31 KEYSW, K32 KEYSW, K33 KEYSW, K34 KEYSW, K35 KEYSW, K36 KEYSW, K41 KEYSW, K44 KEYSW, K45 KEYSW, K46 KEYSW, K51 KEYSW, K54 KEYSW, K55 KEYSW, K56 KEYSW, K61 KEYSW, K65 KEYSW, K66 KEYSW, SW1 SW_PUSH, U1 W25Q128JVS, U2 USBLC6-2SC6, U3 RP2040, U4 XC6206PxxxMR, Y1 XTAL_GND

Commit message: Finalize schematic layout
Parts:
- added D00, D01, D02, D03, D04, D05, D06, D10, D11, D12, D13, D14, D15, D20, D21, D22, D23, D24, D25, D26, D31, D32, D33, D34, D35, D36, D41, D44, D45, D46, D51, D54, D55, D56, D61, D65, D66, D?: D, symbol Device:D
Connections:
- net COL4: now reaches K04.1
- net COL4: now also K14.1, K24.1, K34.1, K44.1, K54.1, U3.6 (GPIO4)
- net at K04.2: now also D04.2 (A)
- net COL2: now reaches K12.1
- net COL2: now also K02.1, K22.1, K32.1, U3.4 (GPIO2)
- net at K12.2: now also D12.2 (A)
- net COL3: now reaches K33.1
- net COL3: now also K03.1, K13.1, K23.1, U3.5 (GPIO3)
- net at K33.2: now also D33.2 (A)
- net COL5: now reaches K25.1
- net COL5: now also K05.1, K15.1, K35.1, K45.1, K55.1, K65.1, U3.7 (GPIO5)
- net at K25.2: now also D25.2 (A)
- net at K45.2: now also D45.2 (A)
- net at K44.2: now also D44.2 (A)
- net COL6: now reaches K36.1
- net COL6: now also K06.1, K26.1, K46.1, K56.1, K66.1, U3.8 (GPIO6)
- net at K36.2: now also D36.2 (A)
- net at K55.2: now also D55.2 (A)
- net COL0: now reaches K10.1
- net COL0: now also K00.1, K20.1, U3.2 (GPIO0)
- net at K10.2: now also D10.2 (A)
- net at K46.2: now also D46.2 (A)
- net at K34.2: now also D34.2 (A)
- net at K54.2: now also D54.2 (A)
- net COL1: now reaches K01.1
- net COL1: now also K11.1, K21.1, K31.1, K41.1, K51.1, K61.1, U3.3 (GPIO1)
- net at K01.2: now also D01.2 (A)
- net at K02.2: now also D02.2 (A)
- net at K65.2: now also D65.2 (A)
- net at K13.2: now also D13.2 (A)
- net at K41.2: now also D41.2 (A)
- net at K06.2: now also D06.2 (A)
- net at K61.2: now also D61.2 (A)
- net at K22.2: now also D22.2 (A)
- net at K31.2: now also D31.2 (A)
- net at K03.2: now also D03.2 (A)
- net at K35.2: now also D35.2 (A)
- net at K15.2: now also D15.2 (A)
- net at K11.2: now also D11.2 (A)
- net at K24.2: now also D24.2 (A)
- net at K00.2: now also D00.2 (A)
- net at K21.2: now also D21.2 (A)
- net at K32.2: now also D32.2 (A)
- net at K05.2: now also D05.2 (A)
- net at K20.2: now also D20.2 (A)
- net at K14.2: now also D14.2 (A)
- net ROW6: now reaches U3.30 (GPIO19)
- net ROW6: now also D61.1 (K), D65.1 (K), D66.1 (K)
- net ROW5: now reaches U3.31 (GPIO20)
- net ROW5: now also D51.1 (K), D54.1 (K), D55.1 (K), D56.1 (K)
- net ROW4: now reaches U3.32 (GPIO21)
- net ROW4: now also D41.1 (K), D44.1 (K), D45.1 (K), D46.1 (K)
- net ROW3: now reaches U3.34 (GPIO22)
- net ROW3: now also D31.1 (K), D32.1 (K), D33.1 (K), D34.1 (K), D35.1 (K), D36.1 (K)
- net ROW2: now reaches U3.35 (GPIO23)
- net ROW2: now also D20.1 (K), D21.1 (K), D22.1 (K), D23.1 (K), D24.1 (K), D25.1 (K), D26.1 (K)
- net ROW1: now reaches U3.36 (GPIO24)
- net ROW1: now also D10.1 (K), D11.1 (K), D12.1 (K), D13.1 (K), D14.1 (K), D15.1 (K)
- net ROW0: now reaches U3.37 (GPIO25)
- net ROW0: now also D00.1 (K), D01.1 (K), D02.1 (K), D03.1 (K), D04.1 (K), D05.1 (K), D06.1 (K)
- net at K26.2: now also D26.2 (A)
- net at K56.2: now also D56.2 (A)
- net at K23.2: now also D23.2 (A)
- net at K66.2: now also D66.2 (A)
- net at K51.2: now also D51.2 (A)
- no-connect marks 4 -> 20
Other:
- moved on the sheet: C4, C7, K00, K01, K02, K03, K04, K05, K06, K10, K11, K12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

Commit message: Schematic finished, started on layout
Parts:
- removed D54, D61, D65, D66, D?: D, symbol Device:D
- removed K54, K61, K65, K66: KEYSW, symbol keyboard_parts:KEYSW
- C1, C10, C11, C12, C13, C14, C2, C3, C4, C5, C6, C7, C8, C9: footprint (none) -> Capacitor_SMD:C_0603_1608Metric
- C15: value 100nF -> 1uF; footprint (none) -> Capacitor_SMD:C_0603_1608Metric
- C16: value 100nF -> 1uF; footprint (none) -> Diode_SMD:D_SOD-123
- D00, D01, D02, D03, D04, D05, D06, D10, D11, D12, D13, D14, D15, D20, D21, D22, D23, D24, D25, D26, D31, D32, D33, D34, D35, D36, D41, D44, D45, D46, D51, D55, D56: footprint (none) -> Diode_SMD:D_SOD-123
- F1: footprint (none) -> Fuse:Fuse_1206_3216Metric
- FID1, FID2, FID3, FID4: footprint (none) -> Fiducial:Fiducial_0.75mm_Mask1.5mm
- J1: footprint (none) -> Connector_USB:USB_C_Receptacle_HRO_TYPE-C-31-M-12
- K00: value KEYSW -> ESC; footprint (none) -> Keeb_Parts:Kailh_MX_Socket
- K01: value KEYSW -> 7; footprint (none) -> Keeb_Parts:Kailh_MX_Socket
- K02: value KEYSW -> 8; footprint (none) -> Keeb_Parts:Kailh_MX_Socket
- K03: value KEYSW -> 9; footprint (none) -> Keeb_Parts:Kailh_MX_Socket
- K04: value KEYSW -> 0; footprint (none) -> Keeb_Parts:Kailh_MX_Socket
- K05: value KEYSW -> -; footprint (none) -> Keeb_Parts:Kailh_MX_Socket
- K06: value KEYSW -> =; footprint (none) -> Keeb_Parts:Kailh_MX_Socket
- K10: value KEYSW -> 1; footprint (none) -> Keeb_Parts:Kailh_MX_Socket
- K11: value KEYSW -> 2; footprint (none) -> Keeb_Parts:Kailh_MX_Socket
- K12: value KEYSW -> 3; footprint (none) -> Keeb_Parts:Kailh_MX_Socket
- K13: value KEYSW -> 4; footprint (none) -> Keeb_Parts:Kailh_MX_Socket
- K14: value KEYSW -> 5; footprint (none) -> Keeb_Parts:Kailh_MX_Socket
- K15: value KEYSW -> 6; footprint (none) -> Keeb_Parts:Kailh_MX_Socket
- K20: value KEYSW -> CAPS; footprint (none) -> Keeb_Parts:Kailh_MX_Socket
- K21: value KEYSW -> TAB; footprint (none) -> Keeb_Parts:Kailh_MX_Socket
- K22: value KEYSW -> Q; footprint (none) -> Keeb_Parts:Kailh_MX_Socket
- K23: value KEYSW -> W; footprint (none) -> Keeb_Parts:Kailh_MX_Socket
- K24: value KEYSW -> E; footprint (none) -> Keeb_Parts:Kailh_MX_Socket
- K25: value KEYSW -> R; footprint (none) -> Keeb_Parts:Kailh_MX_Socket
- K26: value KEYSW -> T; footprint (none) -> Keeb_Parts:Kailh_MX_Socket
- K31: value KEYSW -> LALT; footprint (none) -> Keeb_Parts:Kailh_MX_Socket
- K32: value KEYSW -> A; footprint (none) -> Keeb_Parts:Kailh_MX_Socket
- K33: value KEYSW -> S; footprint (none) -> Keeb_Parts:Kailh_MX_Socket
- K34: value KEYSW -> D; footprint (none) -> Keeb_Parts:Kailh_MX_Socket
- K35: value KEYSW -> F; footprint (none) -> Keeb_Parts:Kailh_MX_Socket
- K36: value KEYSW -> G; footprint (none) -> Keeb_Parts:Kailh_MX_Socket
- K41: value KEYSW -> LSHIFT; footprint (none) -> Keeb_Parts:Kailh_MX_Socket
- K44: value KEYSW -> V; footprint (none) -> Keeb_Parts:Kailh_MX_Socket
- K45: value KEYSW -> B; footprint (none) -> Keeb_Parts:Kailh_MX_Socket
- K46: value KEYSW -> P; footprint (none) -> Keeb_Parts:Kailh_MX_Socket
- K51: value KEYSW -> LCTRL; footprint (none) -> Keeb_Parts:Kailh_MX_Socket
- K55: value KEYSW -> C; footprint (none) -> Keeb_Parts:Kailh_MX_Socket
- K56: value KEYSW -> SPACE; footprint (none) -> Keeb_Parts:Kailh_MX_Socket
- R1, R2, R3, R4, R5, R6, R7: footprint (none) -> Resistor_SMD:R_0603_1608Metric
- SW1: footprint (none) -> Keeb_Parts:SW_TACTILE_SMD
- Y1: footprint (none) -> Crystal:Crystal_SMD_3225-4Pin_3.2x2.5mm
Connections:
- net ~{USB BOOT}: now also R1.1, SW1.2
- net ROW6: no longer names the net of U3.30 (GPIO19)
- net VBUS: no longer names the net of F1.1, J1.A4 (VBUS), J1.A9 (VBUS), J1.B4 (VBUS), J1.B9 (VBUS)
- no-connect marks 20 -> 21
Other:
- moved on the sheet: C4, C7, R1, R2, R5, R6, U3

Commit message: Just a lil updatin'
Parts:
- C16: footprint Diode_SMD:D_SOD-123 -> Capacitor_SMD:C_0603_1608Metric
- U3: footprint Sleep-Lib:RP2040-QFN-56 -> RP2040-QFN:RP2040-QFN-56
- Y1: symbol keyboard_parts:XTAL_GND -> Device:Crystal_GND24
Connections:
- net GND: now also Y1.2, Y1.4; no longer Y1.3
- net XTAL_0: now also Y1.3; no longer Y1.2
- net RESET: no longer names the net of R2.2, U3.26 (~{RUN})
Other:
- moved on the sheet: C2, C3, R7

Commit message: WIP Updates
Parts:
- removed D00, D01, D02, D03, D04, D05, D06, D10, D11, D12, D13, D14, D15, D20, D21, D22, D23, D24, D25, D26, D31, D32, D33, D34, D35, D36, D41, D44, D45, D46, D51, D55, D56: D, Diode_SMD:D_SOD-123, symbol Device:D
- removed FID1, FID2, FID3, FID4: Fiducial, Fiducial:Fiducial_0.75mm_Mask1.5mm, symbol Mechanical:Fiducial
- removed K00: ESC, Keeb_Parts:Kailh_MX_Socket, symbol keyboard_parts:KEYSW
- removed K01: 7, Keeb_Parts:Kailh_MX_Socket, symbol keyboard_parts:KEYSW
- removed K02: 8, Keeb_Parts:Kailh_MX_Socket, symbol keyboard_parts:KEYSW
- removed K03: 9, Keeb_Parts:Kailh_MX_Socket, symbol keyboard_parts:KEYSW
- removed K04: 0, Keeb_Parts:Kailh_MX_Socket, symbol keyboard_parts:KEYSW
- removed K05: -, Keeb_Parts:Kailh_MX_Socket, symbol keyboard_parts:KEYSW
- removed K06: =, Keeb_Parts:Kailh_MX_Socket, symbol keyboard_parts:KEYSW
- removed K10: 1, Keeb_Parts:Kailh_MX_Socket, symbol keyboard_parts:KEYSW
- removed K11: 2, Keeb_Parts:Kailh_MX_Socket, symbol keyboard_parts:KEYSW
- removed K12: 3, Keeb_Parts:Kailh_MX_Socket, symbol keyboard_parts:KEYSW
- removed K13: 4, Keeb_Parts:Kailh_MX_Socket, symbol keyboard_parts:KEYSW
- removed K14: 5, Keeb_Parts:Kailh_MX_Socket, symbol keyboard_parts:KEYSW
- removed K15: 6, Keeb_Parts:Kailh_MX_Socket, symbol keyboard_parts:KEYSW
- removed K20: CAPS, Keeb_Parts:Kailh_MX_Socket, symbol keyboard_parts:KEYSW
- removed K21: TAB, Keeb_Parts:Kailh_MX_Socket, symbol keyboard_parts:KEYSW
- removed K22: Q, Keeb_Parts:Kailh_MX_Socket, symbol keyboard_parts:KEYSW
- removed K23: W, Keeb_Parts:Kailh_MX_Socket, symbol keyboard_parts:KEYSW
- removed K24: E, Keeb_Parts:Kailh_MX_Socket, symbol keyboard_parts:KEYSW
- removed K25: R, Keeb_Parts:Kailh_MX_Socket, symbol keyboard_parts:KEYSW
- removed K26: T, Keeb_Parts:Kailh_MX_Socket, symbol keyboard_parts:KEYSW
- removed K31: LALT, Keeb_Parts:Kailh_MX_Socket, symbol keyboard_parts:KEYSW
- removed K32: A, Keeb_Parts:Kailh_MX_Socket, symbol keyboard_parts:KEYSW
- removed K33: S, Keeb_Parts:Kailh_MX_Socket, symbol keyboard_parts:KEYSW
- removed K34: D, Keeb_Parts:Kailh_MX_Socket, symbol keyboard_parts:KEYSW
- removed K35: F, Keeb_Parts:Kailh_MX_Socket, symbol keyboard_parts:KEYSW
- removed K36: G, Keeb_Parts:Kailh_MX_Socket, symbol keyboard_parts:KEYSW
- removed K41: LSHIFT, Keeb_Parts:Kailh_MX_Socket, symbol keyboard_parts:KEYSW
- removed K44: V, Keeb_Parts:Kailh_MX_Socket, symbol keyboard_parts:KEYSW
- removed K45: B, Keeb_Parts:Kailh_MX_Socket, symbol keyboard_parts:KEYSW
- removed K46: P, Keeb_Parts:Kailh_MX_Socket, symbol keyboard_parts:KEYSW
- removed K51: LCTRL, Keeb_Parts:Kailh_MX_Socket, symbol keyboard_parts:KEYSW
- removed K55: C, Keeb_Parts:Kailh_MX_Socket, symbol keyboard_parts:KEYSW
- removed K56: SPACE, Keeb_Parts:Kailh_MX_Socket, symbol keyboard_parts:KEYSW
- added SW2: SW_PUSH, Keeb_Parts:SW_TACTILE_SMD, symbol keyboard_parts:SW_PUSH
- U3: footprint RP2040-QFN:RP2040-QFN-56 -> Sleep-Lib:RP2040-QFN-56
- renumbered C2 to C1, C3 to C2, C1 to C3
Connections:
- net COL0: now also U3.35 (GPIO23); no longer U3.2 (GPIO0)
- net COL1: now also U3.34 (GPIO22); no longer U3.3 (GPIO1)
- net COL2: now also U3.36 (GPIO24); no longer U3.4 (GPIO2)
- net COL3: now also U3.37 (GPIO25); no longer U3.5 (GPIO3)
- net GND: now also SW2.1
- net ROW0: now also U3.38 (GPIO26/ADC0); no longer U3.37 (GPIO25)
- net ROW1: now also U3.39 (GPIO27/ADC1); no longer U3.36 (GPIO24)
- net ROW2: now also U3.40 (GPIO28/ADC2); no longer U3.35 (GPIO23)
- net ROW3: now also U3.41 (GPIO29/ADC3); no longer U3.34 (GPIO22)
- net at R2.2, U3.26 (~{RUN}): now also SW2.2
Other:
- added sheet SwitchMatrix (switchmatrix.kicad_sch)
- moved on the sheet: C4, C7, R2, R5, R6

Commit message: Ordered JLC Protoparts
Parts:
- C1, C2: MPN (none) -> C1653
- C10, C11, C12, C13, C14, C3, C5, C6, C8, C9: MPN (none) -> C14663
- C15, C16, C4, C7: MPN (none) -> C15849
- F1: MPN (none) -> C70076
- J1: MPN (none) -> C165948
- R1, R2, R7: MPN (none) -> C21190
- R3, R4: MPN (none) -> C23186
- R5, R6: MPN (none) -> C25190
- SW1, SW2: MPN (none) -> C318884
- U1: MPN (none) -> C97521
- U2: MPN (none) -> C85364
- U3: MPN (none) -> C2040
- U4: MPN (none) -> C5446
- Y1: MPN (none) -> C13738
Changed lines of the file:
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@@
+      (effects (font (size 1.27 1.27)) hide)
+    )
+    (property "MPN" "C14663" (id 4) (at 288.544 68.072 0)
       (effects (font (size 1.27 1.27)) hide)
     )
@@
       (effects (font (size 1.27 1.27)) hide)
     )
+    (property "MPN" "C14663" (id 4) (at 280.162 68.072 0)
+      (effects (font (size 1.27 1.27)) hide)
+    )
     (pin "1")
     (pin "2")
@@
       (effects (font (size 1.27 1.27)) hide)
     )
+    (property "MPN" "C25190" (id 4) (at 91.186 44.45 90)
+      (effects (font (size 1.27 1.27)) hide)
+    )
     (pin "1")
     (pin "2")
@@
       (effects (font (size 1.27 1.27)) hide)
     )
+    (property "MPN" "C15849" (id 4) (at 240.284 94.742 0)
+      (effects (font (size 1.27 1.27)) hide)
+    )
     (pin "1")
     (pin "2")
@@
       (effects (font (size 1.27 1.27)) hide)
     )
+    (property "MPN" "C21190" (id 4) (at 192.278 30.988 90)
+      (effects (font (size 1.27 1.27)) hide)
+    )
     (pin "1")
     (pin "2")
@@
       (effects (font (size 1.27 1.27)) hide)
     )
+    (property "MPN" "C15849" (id 4) (at 87.63 68.834 90)
+      (effects (font (size 1.27 1.27)) hide)
+    )
     (pin "1")
     (pin "2")
@@
     )
     (property "Datasheet" "https://www.st.com/resource/en/datasheet/usblc6-2.pdf" (id 3) (at 266.954 23.876 0)
+      (effects (font (size 1.27 1.27)) hide)
+    )
+    (property "MPN" "C85364" (id 4) (at 261.874 32.766 0)
       (effects (font (size 1.27 1.27)) hide)
     )
@@
       (effects (font (size 1.27 1.27)) hide)
     )
+    (property "MPN" "C14663" (id 4) (at 322.072 68.072 0)
+      (effects (font (size 1.27 1.27)) hide)
+    )
     (pin "1")
     (pin "2")
@@
       (effects (font (size 1.27 1.27)) hide)
     )
+    (property "MPN" "C1653" (id 4) (at 301.498 23.622 90)
+      (effects (font (size 1.27 1.27)) hide)
+    )
     (pin "1")
     (pin "2")
@@
       (effects (font (size 1.27 1.27)) hide)
     )
+    (property "MPN" "C25190" (id 4) (at 91.186 41.91 90)
+      (effects (font (size 1.27 1.27)) hide)
+    )
     (pin "1")
     (pin "2")
@@
       (effects (font (size 1.27 1.27)) hide)
     )
+    (property "MPN" "C14663" (id 4) (at 313.69 68.072 0)
+      (effects (font (size 1.27 1.27)) hide)
+    )
     (pin "1")
     (pin "2")
@@
     )
     (property "Datasheet" "~" (id 3) (at 301.498 38.862 0)
+      (effects (font (size 1.27 1.27)) hide)
+    )
+    (property "MPN" "C1653" (id 4) (at 301.498 38.862 90)
       (effects (font (size 1.27 1.27)) hide)
     )
@@
       (effects (font (size 1.524 1.524)))
     )
+    (property "MPN" "C318884" (id 4) (at 84.328 30.48 0)
+      (effects (font (size 1.27 1.27)) hide)
+    )
     (pin "1")
     (pin "2")
@@
       (effects (font (size 1.27 1.27)) hide)
     )
+    (property "MPN" "C14663" (id 4) (at 256.286 68.072 0)
+      (effects (font (size 1.27 1.27)) hide)
+    )
     (pin "1")
     (pin "2")
@@
       (effects (font (size 1.27 1.27)) hide)
     )
+    (property "MPN" "C23186" (id 4) (at 210.82 68.326 90)
+      (effects (font (size 1.27 1.27)) hide)
+    )
     (pin "1")
     (pin "2")
@@
       (effects (font (size 1.27 1.27)) hide)
     )
+    (property "MPN" "C14663" (id 4) (at 246.126 68.072 0)
+      (effects (font (size 1.27 1.27)) hide)
+    )
     (pin "1")
     (pin "2")
@@
       (effects (font (size 1.27 1.27)) hide)
     )
+    (property "MPN" "C14663" (id 4) (at 296.926 68.072 0)
+      (effects (font (size 1.27 1.27)) hide)
+    )
     (pin "1")
     (pin "2")
@@
     )
     (property "Datasheet" "http://www.winbond.com/resource-files/w25q128jv_dtr%20revc%2003272018%20plus.pdf" (id 3) (at 208.788 33.528 0)
+      (effects (font (size 1.27 1.27)) hide)
+    )
+    (property "MPN" "C97521" (id 4) (at 208.788 33.528 0)
       (effects (font (size 1.27 1.27)) hide)
     )
@@
       (effects (font (size 1.27 1.27)) hide)
     )
+    (property "MPN" "C21190" (id 4) (at 91.948 23.114 0)
+      (effects (font (size 1.27 1.27)) hide)
+    )
     (pin "1")
     (pin "2")
@@
     )
     (property "Datasheet" "https://www.usb.org/sites/default/files/documents/usb_type-c.zip" (id 3) (at 188.468 75.946 0)
+      (effects (font (size 1.27 1.27)) hide)
+    )
+    (property "MPN" "C165948" (id 4) (at 184.658 75.946 0)
       (effects (font (size 1.27 1.27)) hide)
     )
@@
       (effects (font (size 1.27 1.27)) hide)
     )
+    (property "MPN" "C23186" (id 4) (at 210.82 65.786 90)
+      (effects (font (size 1.27 1.27)) hide)
+    )
     (pin "1")
     (pin "2")
@@
       (effects (font (size 1.27 1.27)) hide)
     )
+    (property "MPN" "C14663" (id 4) (at 305.308 68.072 0)
+      (effects (font (size 1.27 1.27)) hide)
+    )
     (pin "1")
     (pin "2")
@@
       (effects (font (size 1.27 1.27)) hide)
     )
+    (property "MPN" "C14663" (id 4) (at 271.526 68.072 0)
+      (effects (font (size 1.27 1.27)) hide)
+    )
     (pin "1")
     (pin "2")
@@
     (property "Datasheet" "https://datasheets.raspberrypi.com/rp2040/rp2040-datasheet.pdf" (id 3) (at 97.028 11.43 0)
       (effects (font (size 1.27 1.27)) (justify left bottom) hide)
+    )
+    (property "MPN" "C2040" (id 4) (at 117.348 73.66 0)
+      (effects (font (size 1.27 1.27)) hide)
     )
     (pin "1")
@@
       (effects (font (size 1.27 1.27)) hide)
     )
+    (property "MPN" "C14663" (id 4) (at 217.424 20.066 90)
+      (effects (font (size 1.27 1.27)) hide)
+    )
     (pin "1")
     (pin "2")
@@
     )
     (property "Datasheet" "~" (id 3) (at 312.928 31.242 0)
+      (effects (font (size 1.27 1.27)) hide)
+    )
+    (property "MPN" "C13738" (id 4) (at 312.928 31.242 90)
       (effects (font (size 1.27 1.27)) hide)
     )
@@
     )
     (property "Datasheet" "~" (id 3) (at 86.36 78.74 0)
+      (effects (font (size 1.27 1.27)) hide)
+    )
+    (property "MPN" "C15849" (id 4) (at 86.36 78.74 90)
       (effects (font (size 1.27 1.27)) hide)
     )
@@
       (effects (font (size 1.27 1.27)) hide)
     )
+    (property "MPN" "C70076" (id 4) (at 212.852 60.706 90)
+      (effects (font (size 1.27 1.27)) hide)
+    )
     (pin "1")
     (pin "2")
@@
     )
     (property "Datasheet" "~" (id 3) (at 265.684 94.742 0)
+      (effects (font (size 1.27 1.27)) hide)
+    )
+    (property "MPN" "C15849" (id 4) (at 265.684 94.742 0)
       (effects (font (size 1.27 1.27)) hide)
     )
@@
       (effects (font (size 1.27 1.27)) hide)
     )
+    (property "MPN" "C5446" (id 4) (at 254 88.138 0)
+      (effects (font (size 1.27 1.27)) hide)
+    )
     (pin "1")
     (pin "2")
@@
       (effects (font (size 1.524 1.524)))
     )
+    (property "MPN" "C318884" (id 4) (at 171.704 30.988 0)
+      (effects (font (size 1.27 1.27)) hide)
+    )
     (pin "1")
     (pin "2")
@@
       (effects (font (size 1.27 1.27)) hide)
     )
+    (property "MPN" "C21190" (id 4) (at 330.2 38.862 90)
+      (effects (font (size 1.27 1.27)) hide)
+    )
