File: StealthPad/switchmatrix.kicad_sch (KiCad schematic)
At the start: 66 parts, among them K00 ESC, K01 7, K02 8, K03 9, K04 0, K05 -, K06 =, K10 1, K11 2, K12 3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

Commit message: Ordered JLC Protoparts
Parts:
- D00, D01, D02, D03, D04, D05, D06, D10, D11, D12, D13, D14, D15, D20, D21, D22, D23, D24, D25, D26, D31, D32, D33, D34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: MPN (none) -> C81598
- K00, K01, K02, K03, K04, K05, K06, K10, K11, K12, K13, K14, K15, K20, K21, K22, K23, K24, K25, K26, K31, K32, K33, K34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: MPN (none) -> C5156480
